File: firstm32.kicad_sch (KiCad schematic)
At the start: 36 parts, among them J1 USB_C_Receptacle_USB2.0_16P, J2 Conn_01x04_Pin, J3 Conn_01x04_Pin, J4 Conn_01x04_Pin, SW1 SW_SPDT, U1 AMS1117-3.3, U2 STM32F103C8T6, Y1 16MHz

Commit message: Finished board layout
Parts:
- added H1, H2, H3, H4: MountingHole, MountingHole:MountingHole_2.2mm_M2, symbol Mechanical:MountingHole
Connections:
- net I2C2_SCL: now also J4.2 (Pin_2), R8.1; no longer J4.3 (Pin_3), R7.1
- net I2C2_SDA: now also J4.3 (Pin_3), R7.1; no longer J4.2 (Pin_2), R8.1
Other:
- note added: "HIGH => Bootloader mode LOW => Run-prog mode"
- note added: "Mounting Holes"
